File: KiCad_mini/openradfan.kicad_pcb (KiCad board)
At the start: 2 copper layers, 79.5 x 32 mm, 39 parts, among them CN1 DB141V-2.54-3P, J1 Fan_CPU_4pin, J5 Fan_CPU_4pin, Q1 AO3401A_C347476, U1 74AHCT125, U2 AP63205WU, U3 BTS462TATMA1

Commit message: Prototype fixes
Parts:
- moved TP1 15.2 mm to (46.6, 79.2)
- moved TP2 13.9 mm to (46.6, 72.1)
- moved CN1 12.4 mm to (57.6, 66.5)
- moved J5 8.42 mm to (52.2, 87.2)
- moved J1 8.31 mm to (52.1, 79.0)
- moved TP4 1.50 mm to (87.6, 84.6)
- moved TP3 1.12 mm to (76.1, 83.1)
Routing:
- net PWM_1_BUF: track 14.3 -> 22.6 mm
- net Net-(D2-K): track 9.64 -> 18.0 mm
- net Net-(D1-K): track 14.9 -> 22.6 mm
- net PWM_2_BUF: track 21.2 -> 27.2 mm
- net GPIO_DS18B20: track 34.5 -> 29.0 mm
- net +3.3V: track 44.4 -> 49.2 mm
- net +12V_FAN: track 58.3 -> 62.2 mm

Commit message: Proto rearrangement
Parts:
- moved TP1 60.1 mm to (106.6, 83.7)
- moved H6 19.5 mm to (65.1, 86.1)
- moved TP3 18.4 mm to (80.1, 65.1)
- moved TP4 14.4 mm to (73.6, 81.1)
- moved J1 8.55 mm to (46.6, 85.6), turned to 90 degrees
- moved J5 5.20 mm to (57.1, 85.6), turned to 90 degrees
- moved TP2 1.50 mm to (46.6, 70.6)
Routing:
- net Net-(D2-K): track 18.0 -> 34.3 mm
- net PWM_1_BUF: track 22.6 -> 36.1 mm
- net +12V_FAN: track 62.2 -> 56.6 mm
- net PWM_2_BUF: track 27.2 -> 30.3 mm
- net Net-(D1-K): track 22.6 -> 20.0 mm
- net +5V: track 55.1 -> 52.5 mm
- net +3.3V: track 49.2 -> 48.5 mm
Other:
- board size 79.5 x 32 mm -> 79.5 x 28 mm

Commit message: Tweaks
Parts:
- moved CN1 1.90 mm to (56.5, 68.1), turned to 90 degrees
- moved TP2 1.41 mm to (45.6, 69.6)
- moved H1 0.50 mm to (46.1, 64.6)
Routing:
- net +3.3V: track 48.5 -> 40.6 mm
- net GPIO_DS18B20: track 29.0 -> 29.6 mm
